Commit message: Add materials for chassis and wheels in URDF; enhance Gazebo world with additional models

File: ros2_ws/src/floore_description/urdf/floore.gazebo.xacro (robot description, xacro)
@@ -22,4 +22,42 @@
       <topic>joint_states</topic>
     </plugin>
+  </gazebo>
+  <!-- URDF <material><color> above covers RViz; gz-sim needs its own
+       copy since sdformat's URDF->SDF conversion doesn't reliably carry
+       the URDF material color through to the render engine. -->
+  <gazebo reference="base_link">
+    <material>
+      <ambient>${chassis_color_rgba}</ambient>
+      <diffuse>${chassis_color_rgba}</diffuse>
+      <specular>0.1 0.1 0.1 1</specular>
+    </material>
+  </gazebo>
+  <gazebo reference="front_left_wheel_link">
+    <material>
+      <ambient>${wheel_color_rgba}</ambient>
+      <diffuse>${wheel_color_rgba}</diffuse>
+      <specular>0.1 0.1 0.1 1</specular>
+    </material>
+  </gazebo>
+  <gazebo reference="front_right_wheel_link">
+    <material>
+      <ambient>${wheel_color_rgba}</ambient>
+      <diffuse>${wheel_color_rgba}</diffuse>
+      <specular>0.1 0.1 0.1 1</specular>
+    </material>
+  </gazebo>
+  <gazebo reference="rear_left_wheel_link">
+    <material>
+      <ambient>${wheel_color_rgba}</ambient>
+      <diffuse>${wheel_color_rgba}</diffuse>
+      <specular>0.1 0.1 0.1 1</specular>
+    </material>
+  </gazebo>
+  <gazebo reference="rear_right_wheel_link">
+    <material>
+      <ambient>${wheel_color_rgba}</ambient>
+      <diffuse>${wheel_color_rgba}</diffuse>
+      <specular>0.1 0.1 0.1 1</specular>
+    </material>
   </gazebo>
   <!-- 2D LiDAR. type=gpu_lidar requires the world-level Sensors system

File: ros2_ws/src/floore_description/urdf/floore.urdf.xacro (robot description, xacro)
@@ -43,4 +43,6 @@
   <xacro:property name="chassis_mass" value="8.0"/>
   <xacro:property name="wheel_mass" value="0.3"/>
+  <xacro:property name="chassis_color_rgba" value="0.85 0.65 0.13 1.0"/>
+  <xacro:property name="wheel_color_rgba" value="0.15 0.15 0.15 1.0"/>
   <!-- ============================================================
        base_link / chassis. base_link IS the chassis mesh's native
@@ -54,4 +56,7 @@
         <mesh filename="package://floore_description/meshes/collision/Chassis.STL" scale="${mesh_scale}"/>
       </geometry>
+      <material name="chassis_yellow">
+        <color rgba="${chassis_color_rgba}"/>
+      </material>
     </visual>
     <collision>
@@ -86,4 +91,7 @@
           <mesh filename="package://floore_description/meshes/collision/${mesh_file}" scale="${mesh_scale}"/>
         </geometry>
+        <material name="wheel_dark_grey">
+          <color rgba="${wheel_color_rgba}"/>
+        </material>
       </visual>
       <collision>
